File: mbed_lpc1114.kicad_pcb (KiCad board)
At the start: 2 copper layers, 100 x 100 mm, 32 parts, among them J1 CONN_01X01, J10 CONN_01X01, J11 CONN_01X01, J12 CONN_01X01, J13 CONN_01X01, J14 CONN_01X01, J15 CONN_01X01, J16 CONN_01X01, J17 CONN_01X01, J18 CONN_01X01, J19 CONN_01X01, J2 CONN_01X01, J20 CONN_01X01, J21 CONN_01X01, J22 CONN_01X01, J23 CONN_01X06, J24 BARREL_JACK, J3 CONN_01X01, J4 CONN_01X01, J5 CONN_01X01, J6 CONN_01X01, J7 CONN_01X01, J8 CONN_01X01, J9 CONN_01X01, U1 7803, U2 lpc1114fn28

Commit message: 完成
Parts:
- added ?: , pad:universal, F.Cu at (143.5, 125.1)
- added ?: , pad:universal, F.Cu at (123.2, 125.1)
- added ?: , pad:universal, F.Cu at (87.6, 89.5)
- added ?: , pad:universal, F.Cu at (181.6, 130.2)
- added ?: , pad:universal, F.Cu at (166.4, 130.2)
- added ?: , pad:universal, F.Cu at (166.4, 132.7)
- added ?: , pad:universal, F.Cu at (163.8, 132.7)
- added ?: , pad:universal, F.Cu at (163.8, 130.2)
- added ?: , pad:universal, F.Cu at (171.4, 132.7)
- added ?: , pad:universal, F.Cu at (171.4, 130.2)
- added ?: , pad:universal, F.Cu at (168.9, 132.7)
- added ?: , pad:universal, F.Cu at (168.9, 130.2)
- added ?: , pad:universal, F.Cu at (151.1, 132.7)
- added ?: , pad:universal, F.Cu at (90.2, 89.5)
- added ?: , pad:universal, F.Cu at (148.6, 130.2)
- added ?: , pad:universal, F.Cu at (148.6, 132.7)
- added ?: , pad:universal, F.Cu at (151.1, 130.2)
- added ?: , pad:universal, F.Cu at (158.8, 130.2)
- added ?: , pad:universal, F.Cu at (161.3, 132.7)
- added ?: , pad:universal, F.Cu at (158.8, 132.7)
- added ?: , pad:universal, F.Cu at (161.3, 130.2)
- added ?: , pad:universal, F.Cu at (163.8, 120.0)
- added ?: , pad:universal, F.Cu at (166.4, 122.6)
- added ?: , pad:universal, F.Cu at (166.4, 120.0)
- added ?: , pad:universal, F.Cu at (92.7, 89.5)
- added ?: , pad:universal, F.Cu at (163.8, 122.6)
- added ?: , pad:universal, F.Cu at (176.5, 122.6)
- added ?: , pad:universal, F.Cu at (179.1, 122.6)
- added ?: , pad:universal, F.Cu at (176.5, 120.0)
- added ?: , pad:universal, F.Cu at (179.1, 120.0)
- added ?: , pad:universal, F.Cu at (168.9, 120.0)
- added ?: , pad:universal, F.Cu at (171.4, 120.0)
- added ?: , pad:universal, F.Cu at (171.4, 122.6)
- added ?: , pad:universal, F.Cu at (168.9, 122.6)
- added ?: , pad:universal, F.Cu at (174.0, 122.6)
- added ?: , pad:universal, F.Cu at (95.2, 92.1)
- added ?: , pad:universal, F.Cu at (181.6, 120.0)
- added ?: , pad:universal, F.Cu at (181.6, 122.6)
- added ?: , pad:universal, F.Cu at (174.0, 120.0)
- added ?: , pad:universal, F.Cu at (161.3, 120.0)
- added ?: , pad:universal, F.Cu at (151.1, 122.6)
- added ?: , pad:universal, F.Cu at (153.7, 122.6)
- added ?: , pad:universal, F.Cu at (148.6, 122.6)
- added ?: , pad:universal, F.Cu at (153.7, 120.0)
- added ?: , pad:universal, F.Cu at (148.6, 120.0)
- added ?: , pad:universal, F.Cu at (151.1, 120.0)
- added ?: , pad:universal, F.Cu at (95.2, 89.5)
- added ?: , pad:universal, F.Cu at (158.8, 122.6)
- added ?: , pad:universal, F.Cu at (158.8, 120.0)
- added ?: , pad:universal, F.Cu at (156.2, 122.6)
- added ?: , pad:universal, F.Cu at (156.2, 120.0)
- added ?: , pad:universal, F.Cu at (161.3, 122.6)
- added ?: , pad:universal, F.Cu at (158.8, 127.6)
- added ?: , pad:universal, F.Cu at (158.8, 125.1)
- added ?: , pad:universal, F.Cu at (153.7, 125.1)
- added ?: , pad:universal, F.Cu at (156.2, 125.1)
- added ?: , pad:universal, F.Cu at (156.2, 127.6)
- added ?: , pad:universal, F.Cu at (100.3, 89.5)
- added ?: , pad:universal, F.Cu at (168.9, 127.6)
- added ?: , pad:universal, F.Cu at (163.8, 127.6)
- added ?: , pad:universal, F.Cu at (163.8, 125.1)
- added ?: , pad:universal, F.Cu at (166.4, 125.1)
- added ?: , pad:universal, F.Cu at (161.3, 127.6)
- added ?: , pad:universal, F.Cu at (166.4, 127.6)
- added ?: , pad:universal, F.Cu at (161.3, 125.1)
- added ?: , pad:universal, F.Cu at (168.9, 125.1)
- added ?: , pad:universal, F.Cu at (171.4, 125.1)
- added ?: , pad:universal, F.Cu at (174.0, 125.1)
- added ?: , pad:universal, F.Cu at (97.8, 89.5)
- added ?: , pad:universal, F.Cu at (174.0, 127.6)
- added ?: , pad:universal, F.Cu at (171.4, 127.6)
- added ?: , pad:universal, F.Cu at (148.6, 127.6)
- added ?: , pad:universal, F.Cu at (151.1, 125.1)
- added ?: , pad:universal, F.Cu at (151.1, 127.6)
- added ?: , pad:universal, F.Cu at (153.7, 127.6)
- added ?: , pad:universal, F.Cu at (148.6, 125.1)
- added ?: , pad:universal, F.Cu at (181.6, 125.1)
- added ?: , pad:universal, F.Cu at (179.1, 125.1)
- added ?: , pad:universal, F.Cu at (176.5, 127.6)
- added ?: , pad:universal, F.Cu at (100.3, 92.1)
- added ?: , pad:universal, F.Cu at (179.1, 127.6)
- added ?: , pad:universal, F.Cu at (181.6, 127.6)
- added ?: , pad:universal, F.Cu at (176.5, 125.1)
- added ?: , pad:universal, F.Cu at (181.6, 114.9)
- added ?: , pad:universal, F.Cu at (179.1, 114.9)
- added ?: , pad:universal, F.Cu at (176.5, 117.5)
- added ?: , pad:universal, F.Cu at (179.1, 117.5)
- added ?: , pad:universal, F.Cu at (181.6, 117.5)
- added ?: , pad:universal, F.Cu at (176.5, 114.9)
- added ?: , pad:universal, F.Cu at (171.4, 117.5)
- added ?: , pad:universal, F.Cu at (92.7, 92.1)
- added ?: , pad:universal, F.Cu at (168.9, 117.5)
- added ?: , pad:universal, F.Cu at (168.9, 114.9)
- added ?: , pad:universal, F.Cu at (171.4, 114.9)
- added ?: , pad:universal, F.Cu at (174.0, 114.9)
- added ?: , pad:universal, F.Cu at (174.0, 117.5)
- added ?: , pad:universal, F.Cu at (161.3, 117.5)
- added ?: , pad:universal, F.Cu at (163.8, 117.5)
- added ?: , pad:universal, F.Cu at (158.8, 117.5)
- added ?: , pad:universal, F.Cu at (166.4, 117.5)
- added ?: , pad:universal, F.Cu at (158.8, 114.9)
- added ?: , pad:universal, F.Cu at (87.6, 92.1)
- added ?: , pad:universal, F.Cu at (161.3, 114.9)
- added ?: , pad:universal, F.Cu at (163.8, 114.9)
- added ?: , pad:universal, F.Cu at (166.4, 114.9)
- added ?: , pad:universal, F.Cu at (148.6, 117.5)
- added ?: , pad:universal, F.Cu at (151.1, 114.9)
- added ?: , pad:universal, F.Cu at (153.7, 114.9)
- added ?: , pad:universal, F.Cu at (156.2, 114.9)
- added ?: , pad:universal, F.Cu at (156.2, 117.5)
- added ?: , pad:universal, F.Cu at (151.1, 117.5)
- added ?: , pad:universal, F.Cu at (153.7, 117.5)
- added ?: , pad:universal, F.Cu at (138.4, 127.6)
- added ?: , pad:universal, F.Cu at (90.2, 92.1)
- added ?: , pad:universal, F.Cu at (148.6, 114.9)
- added ?: , pad:universal, F.Cu at (161.3, 112.4)
- added ?: , pad:universal, F.Cu at (158.8, 112.4)
- added ?: , pad:universal, F.Cu at (148.6, 112.4)
- added ?: , pad:universal, F.Cu at (151.1, 112.4)
- added ?: , pad:universal, F.Cu at (153.7, 112.4)
- added ?: , pad:universal, F.Cu at (156.2, 112.4)
- added ?: , pad:universal, F.Cu at (181.6, 109.9)
- added ?: , pad:universal, F.Cu at (179.1, 109.9)
- added ?: , pad:universal, F.Cu at (171.4, 112.4)
- added ?: , pad:universal, F.Cu at (110.5, 89.5)
- added ?: , pad:universal, F.Cu at (163.8, 112.4)
- added ?: , pad:universal, F.Cu at (166.4, 112.4)
- added ?: , pad:universal, F.Cu at (168.9, 112.4)
- added ?: , pad:universal, F.Cu at (181.6, 112.4)
- added ?: , pad:universal, F.Cu at (174.0, 112.4)
- added ?: , pad:universal, F.Cu at (176.5, 112.4)
- added ?: , pad:universal, F.Cu at (179.1, 112.4)
- added ?: , pad:universal, F.Cu at (176.5, 109.9)
- added ?: , pad:universal, F.Cu at (168.9, 109.9)
- added ?: , pad:universal, F.Cu at (171.4, 109.9)
- added ?: , pad:universal, F.Cu at (110.5, 92.1)
- added ?: , pad:universal, F.Cu at (174.0, 109.9)
- added ?: , pad:universal, F.Cu at (166.4, 109.9)
- added ?: , pad:universal, F.Cu at (158.8, 109.9)
- added ?: , pad:universal, F.Cu at (161.3, 109.9)
- added ?: , pad:universal, F.Cu at (163.8, 109.9)
- added ?: , pad:universal, F.Cu at (156.2, 109.9)
- added ?: , pad:universal, F.Cu at (148.6, 109.9)
- added ?: , pad:universal, F.Cu at (151.1, 109.9)
- added ?: , pad:universal, F.Cu at (153.7, 109.9)
- added ?: , pad:universal, F.Cu at (108.0, 89.5)
- added ?: , pad:universal, F.Cu at (108.0, 92.1)
- added ?: , pad:universal, F.Cu at (118.1, 92.1)
- added ?: , pad:universal, F.Cu at (120.7, 92.1)
- added ?: , pad:universal, F.Cu at (120.7, 89.5)
- added ?: , pad:universal, F.Cu at (118.1, 89.5)
- added ?: , pad:universal, F.Cu at (102.9, 92.1)
- added ?: , pad:universal, F.Cu at (138.4, 132.7)
- added ?: , pad:universal, F.Cu at (102.9, 89.5)
- added ?: , pad:universal, F.Cu at (105.4, 92.1)
- added ?: , pad:universal, F.Cu at (105.4, 89.5)
- added ?: , pad:universal, F.Cu at (113.0, 89.5)
- added ?: , pad:universal, F.Cu at (113.0, 92.1)
- added ?: , pad:universal, F.Cu at (115.6, 92.1)
- added ?: , pad:universal, F.Cu at (115.6, 89.5)
- added ?: , pad:universal, F.Cu at (168.9, 168.3)
- added ?: , pad:universal, F.Cu at (166.4, 168.3)
- added ?: , pad:universal, F.Cu at (168.9, 170.8)
- added ?: , pad:universal, F.Cu at (138.4, 130.2)
- added ?: , pad:universal, F.Cu at (166.4, 170.8)
- added ?: , pad:universal, F.Cu at (168.9, 173.4)
- added ?: , pad:universal, F.Cu at (166.4, 173.4)
- added ?: , pad:universal, F.Cu at (174.0, 173.4)
- added ?: , pad:universal, F.Cu at (171.4, 170.8)
- added ?: , pad:universal, F.Cu at (171.4, 173.4)
- added ?: , pad:universal, F.Cu at (171.4, 168.3)
- added ?: , pad:universal, F.Cu at (174.0, 170.8)
- added ?: , pad:universal, F.Cu at (174.0, 168.3)
- added ?: , pad:universal, F.Cu at (146.1, 168.3)
- added ?: , pad:universal, F.Cu at (141.0, 130.2)
- added ?: , pad:universal, F.Cu at (146.1, 173.4)
- added ?: , pad:universal, F.Cu at (148.6, 173.4)
- added ?: , pad:universal, F.Cu at (146.1, 170.8)
- added ?: , pad:universal, F.Cu at (143.5, 173.4)
- added ?: , pad:universal, F.Cu at (148.6, 168.3)
- added ?: , pad:universal, F.Cu at (148.6, 170.8)
- added ?: , pad:universal, F.Cu at (133.3, 173.4)
- added ?: , pad:universal, F.Cu at (135.9, 168.3)
- added ?: , pad:universal, F.Cu at (133.3, 170.8)
- added ?: , pad:universal, F.Cu at (135.9, 170.8)
- added ?: , pad:universal, F.Cu at (141.0, 132.7)
- added ?: , pad:universal, F.Cu at (138.4, 173.4)
- added ?: , pad:universal, F.Cu at (133.3, 168.3)
- added ?: , pad:universal, F.Cu at (138.4, 170.8)
- added ?: , pad:universal, F.Cu at (135.9, 173.4)
- added ?: , pad:universal, F.Cu at (138.4, 168.3)
- added ?: , pad:universal, F.Cu at (141.0, 173.4)
- added ?: , pad:universal, F.Cu at (141.0, 168.3)
- added ?: , pad:universal, F.Cu at (143.5, 168.3)
- added ?: , pad:universal, F.Cu at (143.5, 170.8)
- added ?: , pad:universal, F.Cu at (141.0, 170.8)
- added ?: , pad:universal, F.Cu at (141.0, 127.6)
- added ?: , pad:universal, F.Cu at (158.8, 170.8)
- added ?: , pad:universal, F.Cu at (161.3, 168.3)
- added ?: , pad:universal, F.Cu at (158.8, 173.4)
- added ?: , pad:universal, F.Cu at (158.8, 168.3)
- added ?: , pad:universal, F.Cu at (151.1, 173.4)
- added ?: , pad:universal, F.Cu at (156.2, 173.4)
- added ?: , pad:universal, F.Cu at (153.7, 170.8)
- added ?: , pad:universal, F.Cu at (151.1, 170.8)
- added ?: , pad:universal, F.Cu at (153.7, 173.4)
- added ?: , pad:universal, F.Cu at (156.2, 170.8)
- added ?: , pad:universal, F.Cu at (135.9, 127.6)
- added ?: , pad:universal, F.Cu at (151.1, 168.3)
- added ?: , pad:universal, F.Cu at (156.2, 168.3)
- added ?: , pad:universal, F.Cu at (153.7, 168.3)
- added ?: , pad:universal, F.Cu at (163.8, 173.4)
- added ?: , pad:universal, F.Cu at (161.3, 173.4)
- added ?: , pad:universal, F.Cu at (163.8, 170.8)
- added ?: , pad:universal, F.Cu at (161.3, 170.8)
- added ?: , pad:universal, F.Cu at (163.8, 168.3)
- added ?: , pad:universal, F.Cu at (95.2, 168.3)
- added ?: , pad:universal, F.Cu at (97.8, 168.3)
- added ?: , pad:universal, F.Cu at (133.3, 132.7)
- added ?: , pad:universal, F.Cu at (95.2, 170.8)
- added ?: , pad:universal, F.Cu at (97.8, 170.8)
- added ?: , pad:universal, F.Cu at (97.8, 173.4)
- added ?: , pad:universal, F.Cu at (95.2, 173.4)
- added ?: , pad:universal, F.Cu at (113.0, 173.4)
- added ?: , pad:universal, F.Cu at (113.0, 170.8)
- added ?: , pad:universal, F.Cu at (115.6, 170.8)
- added ?: , pad:universal, F.Cu at (115.6, 173.4)
- added ?: , pad:universal, F.Cu at (115.6, 168.3)
- added ?: , pad:universal, F.Cu at (113.0, 168.3)
- added ?: , pad:universal, F.Cu at (133.3, 130.2)
- added ?: , pad:universal, F.Cu at (110.5, 168.3)
- added ?: , pad:universal, F.Cu at (108.0, 168.3)
- added ?: , pad:universal, F.Cu at (105.4, 168.3)
- added ?: , pad:universal, F.Cu at (110.5, 170.8)
- added ?: , pad:universal, F.Cu at (105.4, 173.4)
- added ?: , pad:universal, F.Cu at (105.4, 170.8)
- added ?: , pad:universal, F.Cu at (110.5, 173.4)
- added ?: , pad:universal, F.Cu at (108.0, 173.4)
- added ?: , pad:universal, F.Cu at (108.0, 170.8)
- added ?: , pad:universal, F.Cu at (102.9, 173.4)
- added ?: , pad:universal, F.Cu at (146.1, 125.1)
- added ?: , pad:universal, F.Cu at (135.9, 130.2)
- added ?: , pad:universal, F.Cu at (100.3, 170.8)
- added ?: , pad:universal, F.Cu at (102.9, 170.8)
- added ?: , pad:universal, F.Cu at (100.3, 173.4)
- added ?: , pad:universal, F.Cu at (100.3, 168.3)
- added ?: , pad:universal, F.Cu at (102.9, 168.3)
- added ?: , pad:universal, F.Cu at (118.1, 170.8)
- added ?: , pad:universal, F.Cu at (120.7, 170.8)
- added ?: , pad:universal, F.Cu at (118.1, 173.4)
- added ?: , pad:universal, F.Cu at (123.2, 173.4)
- added ?: , pad:universal, F.Cu at (120.7, 173.4)
- added ?: , pad:universal, F.Cu at (135.9, 132.7)
- added ?: , pad:universal, F.Cu at (130.8, 170.8)
- added ?: , pad:universal, F.Cu at (130.8, 173.4)
- added ?: , pad:universal, F.Cu at (125.7, 170.8)
- added ?: , pad:universal, F.Cu at (128.3, 173.4)
- added ?: , pad:universal, F.Cu at (128.3, 170.8)
- added ?: , pad:universal, F.Cu at (125.7, 173.4)
- added ?: , pad:universal, F.Cu at (118.1, 168.3)
- added ?: , pad:universal, F.Cu at (120.7, 168.3)
- added ?: , pad:universal, F.Cu at (123.2, 168.3)
- added ?: , pad:universal, F.Cu at (123.2, 170.8)
- added ?: , pad:universal, F.Cu at (133.3, 127.6)
- added ?: , pad:universal, F.Cu at (130.8, 168.3)
- added ?: , pad:universal, F.Cu at (125.7, 168.3)
- added ?: , pad:universal, F.Cu at (128.3, 168.3)
- added ?: , pad:universal, F.Cu at (97.8, 158.1)
- added ?: , pad:universal, F.Cu at (95.2, 158.1)
- added ?: , pad:universal, F.Cu at (95.2, 160.7)
- added ?: , pad:universal, F.Cu at (97.8, 160.7)
- added ?: , pad:universal, F.Cu at (90.2, 160.7)
- added ?: , pad:universal, F.Cu at (92.7, 160.7)
- added ?: , pad:universal, F.Cu at (87.6, 158.1)
- added ?: , pad:universal, F.Cu at (128.3, 127.6)
- added ?: , pad:universal, F.Cu at (87.6, 160.7)
- added ?: , pad:universal, F.Cu at (90.2, 158.1)
- added ?: , pad:universal, F.Cu at (92.7, 158.1)
- added ?: , pad:universal, F.Cu at (92.7, 163.2)
- added ?: , pad:universal, F.Cu at (87.6, 163.2)
- added ?: , pad:universal, F.Cu at (90.2, 163.2)
- added ?: , pad:universal, F.Cu at (95.2, 163.2)
- added ?: , pad:universal, F.Cu at (95.2, 165.7)
- added ?: , pad:universal, F.Cu at (97.8, 163.2)
- added ?: , pad:universal, F.Cu at (97.8, 165.7)
- added ?: , pad:universal, F.Cu at (130.8, 130.2)
- added ?: , pad:universal, F.Cu at (115.6, 160.7)
- added ?: , pad:universal, F.Cu at (115.6, 158.1)
- added ?: , pad:universal, F.Cu at (118.1, 158.1)
- added ?: , pad:universal, F.Cu at (118.1, 160.7)
- added ?: , pad:universal, F.Cu at (115.6, 165.7)
- added ?: , pad:universal, F.Cu at (118.1, 165.7)
- added ?: , pad:universal, F.Cu at (115.6, 163.2)
- added ?: , pad:universal, F.Cu at (118.1, 163.2)
- added ?: , pad:universal, F.Cu at (113.0, 165.7)
- added ?: , pad:universal, F.Cu at (113.0, 163.2)
- added ?: , pad:universal, F.Cu at (130.8, 132.7)
- added ?: , pad:universal, F.Cu at (113.0, 160.7)
- added ?: , pad:universal, F.Cu at (110.5, 158.1)
- added ?: , pad:universal, F.Cu at (113.0, 158.1)
- added ?: , pad:universal, F.Cu at (110.5, 160.7)
- added ?: , pad:universal, F.Cu at (108.0, 163.2)
- added ?: , pad:universal, F.Cu at (110.5, 165.7)
- added ?: , pad:universal, F.Cu at (110.5, 163.2)
- added ?: , pad:universal, F.Cu at (105.4, 165.7)
- added ?: , pad:universal, F.Cu at (105.4, 163.2)
- added ?: , pad:universal, F.Cu at (102.9, 165.7)
- added ?: , pad:universal, F.Cu at (128.3, 130.2)
- added ?: , pad:universal, F.Cu at (108.0, 165.7)
- added ?: , pad:universal, F.Cu at (100.3, 163.2)
- added ?: , pad:universal, F.Cu at (100.3, 165.7)
- added ?: , pad:universal, F.Cu at (102.9, 163.2)
- added ?: , pad:universal, F.Cu at (100.3, 160.7)
- added ?: , pad:universal, F.Cu at (100.3, 158.1)
- added ?: , pad:universal, F.Cu at (102.9, 158.1)
- added ?: , pad:universal, F.Cu at (102.9, 160.7)
- added ?: , pad:universal, F.Cu at (105.4, 158.1)
- added ?: , pad:universal, F.Cu at (108.0, 160.7)
- added ?: , pad:universal, F.Cu at (130.8, 127.6)
- added ?: , pad:universal, F.Cu at (105.4, 160.7)
- added ?: , pad:universal, F.Cu at (108.0, 158.1)
- added ?: , pad:universal, F.Cu at (133.3, 165.7)
- added ?: , pad:universal, F.Cu at (133.3, 160.7)
- added ?: , pad:universal, F.Cu at (133.3, 163.2)
- added ?: , pad:universal, F.Cu at (130.8, 163.2)
- added ?: , pad:universal, F.Cu at (130.8, 160.7)
- added ?: , pad:universal, F.Cu at (128.3, 160.7)
- added ?: , pad:universal, F.Cu at (125.7, 163.2)
- added ?: , pad:universal, F.Cu at (125.7, 160.7)
- added ?: , pad:universal, F.Cu at (123.2, 127.6)
- added ?: , pad:universal, F.Cu at (123.2, 160.7)
- added ?: , pad:universal, F.Cu at (120.7, 160.7)
- added ?: , pad:universal, F.Cu at (130.8, 158.1)
- added ?: , pad:universal, F.Cu at (128.3, 158.1)
- added ?: , pad:universal, F.Cu at (120.7, 158.1)
- added ?: , pad:universal, F.Cu at (125.7, 158.1)
- added ?: , pad:universal, F.Cu at (123.2, 158.1)
- added ?: , pad:universal, F.Cu at (120.7, 163.2)
- added ?: , pad:universal, F.Cu at (123.2, 163.2)
- added ?: , pad:universal, F.Cu at (120.7, 165.7)
- added ?: , pad:universal, F.Cu at (125.7, 127.6)
- added ?: , pad:universal, F.Cu at (123.2, 165.7)
- added ?: , pad:universal, F.Cu at (130.8, 165.7)
- added ?: , pad:universal, F.Cu at (125.7, 165.7)
- added ?: , pad:universal, F.Cu at (128.3, 163.2)
- added ?: , pad:universal, F.Cu at (128.3, 165.7)
- added ?: , pad:universal, F.Cu at (174.0, 165.7)
- added ?: , pad:universal, F.Cu at (171.4, 163.2)
- added ?: , pad:universal, F.Cu at (171.4, 165.7)
- added ?: , pad:universal, F.Cu at (171.4, 160.7)
- added ?: , pad:universal, F.Cu at (168.9, 160.7)
- added ?: , pad:universal, F.Cu at (138.4, 125.1)
- added ?: , pad:universal, F.Cu at (125.7, 130.2)
- added ?: , pad:universal, F.Cu at (176.5, 158.1)
- added ?: , pad:universal, F.Cu at (174.0, 158.1)
- added ?: , pad:universal, F.Cu at (166.4, 165.7)
- added ?: , pad:universal, F.Cu at (168.9, 163.2)
- added ?: , pad:universal, F.Cu at (166.4, 160.7)
- added ?: , pad:universal, F.Cu at (166.4, 163.2)
- added ?: , pad:universal, F.Cu at (168.9, 165.7)
- added ?: , pad:universal, F.Cu at (174.0, 163.2)
- added ?: , pad:universal, F.Cu at (176.5, 163.2)
- added ?: , pad:universal, F.Cu at (174.0, 160.7)
- added ?: , pad:universal, F.Cu at (123.2, 132.7)
- added ?: , pad:universal, F.Cu at (179.1, 163.2)
- added ?: , pad:universal, F.Cu at (179.1, 160.7)
- added ?: , pad:universal, F.Cu at (181.6, 160.7)
- added ?: , pad:universal, F.Cu at (176.5, 160.7)
- added ?: , pad:universal, F.Cu at (181.6, 163.2)
- added ?: , pad:universal, F.Cu at (181.6, 158.1)
- added ?: , pad:universal, F.Cu at (179.1, 158.1)
- added ?: , pad:universal, F.Cu at (168.9, 158.1)
- added ?: , pad:universal, F.Cu at (171.4, 158.1)
- added ?: , pad:universal, F.Cu at (166.4, 158.1)
- added ?: , pad:universal, F.Cu at (125.7, 132.7)
- added ?: , pad:universal, F.Cu at (163.8, 158.1)
- added ?: , pad:universal, F.Cu at (151.1, 160.7)
- added ?: , pad:universal, F.Cu at (151.1, 158.1)
- added ?: , pad:universal, F.Cu at (146.1, 160.7)
- added ?: , pad:universal, F.Cu at (148.6, 160.7)
- added ?: , pad:universal, F.Cu at (148.6, 158.1)
- added ?: , pad:universal, F.Cu at (146.1, 158.1)
- added ?: , pad:universal, F.Cu at (146.1, 165.7)
- added ?: , pad:universal, F.Cu at (148.6, 165.7)
- added ?: , pad:universal, F.Cu at (151.1, 165.7)
- added ?: , pad:universal, F.Cu at (128.3, 132.7)
- added ?: , pad:universal, F.Cu at (153.7, 163.2)
- added ?: , pad:universal, F.Cu at (146.1, 163.2)
- added ?: , pad:universal, F.Cu at (151.1, 163.2)
- added ?: , pad:universal, F.Cu at (148.6, 163.2)
- added ?: , pad:universal, F.Cu at (153.7, 165.7)
- added ?: , pad:universal, F.Cu at (163.8, 165.7)
- added ?: , pad:universal, F.Cu at (158.8, 163.2)
- added ?: , pad:universal, F.Cu at (158.8, 165.7)
- added ?: , pad:universal, F.Cu at (158.8, 160.7)
- added ?: , pad:universal, F.Cu at (161.3, 165.7)
- added ?: , pad:universal, F.Cu at (123.2, 130.2)
- added ?: , pad:universal, F.Cu at (163.8, 163.2)
- added ?: , pad:universal, F.Cu at (161.3, 158.1)
- added ?: , pad:universal, F.Cu at (163.8, 160.7)
- added ?: , pad:universal, F.Cu at (161.3, 160.7)
- added ?: , pad:universal, F.Cu at (161.3, 163.2)
- added ?: , pad:universal, F.Cu at (156.2, 163.2)
- added ?: , pad:universal, F.Cu at (156.2, 165.7)
- added ?: , pad:universal, F.Cu at (158.8, 158.1)
- added ?: , pad:universal, F.Cu at (156.2, 160.7)
- added ?: , pad:universal, F.Cu at (153.7, 158.1)
- added ?: , pad:universal, F.Cu at (123.2, 135.3)
- added ?: , pad:universal, F.Cu at (156.2, 158.1)
- added ?: , pad:universal, F.Cu at (153.7, 160.7)
- added ?: , pad:universal, F.Cu at (135.9, 160.7)
- added ?: , pad:universal, F.Cu at (138.4, 160.7)
- added ?: , pad:universal, F.Cu at (138.4, 158.1)
- added ?: , pad:universal, F.Cu at (133.3, 158.1)
- added ?: , pad:universal, F.Cu at (135.9, 158.1)
- added ?: , pad:universal, F.Cu at (141.0, 165.7)
- added ?: , pad:universal, F.Cu at (135.9, 163.2)
- added ?: , pad:universal, F.Cu at (143.5, 165.7)
- added ?: , pad:universal, F.Cu at (123.2, 137.8)
- added ?: , pad:universal, F.Cu at (143.5, 163.2)
- added ?: , pad:universal, F.Cu at (138.4, 165.7)
- added ?: , pad:universal, F.Cu at (141.0, 163.2)
- added ?: , pad:universal, F.Cu at (135.9, 165.7)
- added ?: , pad:universal, F.Cu at (138.4, 163.2)
- added ?: , pad:universal, F.Cu at (141.0, 160.7)
- added ?: , pad:universal, F.Cu at (141.0, 158.1)
- added ?: , pad:universal, F.Cu at (143.5, 160.7)
- added ?: , pad:universal, F.Cu at (143.5, 158.1)
- added ?: , pad:universal, F.Cu at (120.7, 94.6)
- added ?: , pad:universal, F.Cu at (123.2, 140.3)
- added ?: , pad:universal, F.Cu at (115.6, 97.2)
- added ?: , pad:universal, F.Cu at (118.1, 97.2)
- added ?: , pad:universal, F.Cu at (118.1, 94.6)
- added ?: , pad:universal, F.Cu at (115.6, 94.6)
- added ?: , pad:universal, F.Cu at (87.6, 107.3)
- added ?: , pad:universal, F.Cu at (95.2, 107.3)
- added ?: , pad:universal, F.Cu at (90.2, 107.3)
- added ?: , pad:universal, F.Cu at (92.7, 104.8)
- added ?: , pad:universal, F.Cu at (97.8, 107.3)
- added ?: , pad:universal, F.Cu at (92.7, 107.3)
- added ?: , pad:universal, F.Cu at (125.7, 135.3)
- added ?: , pad:universal, F.Cu at (95.2, 104.8)
- added ?: , pad:universal, F.Cu at (90.2, 104.8)
- added ?: , pad:universal, F.Cu at (97.8, 104.8)
- added ?: , pad:universal, F.Cu at (90.2, 102.2)
- added ?: , pad:universal, F.Cu at (87.6, 102.2)
- added ?: , pad:universal, F.Cu at (90.2, 99.7)
- added ?: , pad:universal, F.Cu at (87.6, 99.7)
- added ?: , pad:universal, F.Cu at (87.6, 104.8)
- added ?: , pad:universal, F.Cu at (97.8, 102.2)
- added ?: , pad:universal, F.Cu at (92.7, 102.2)
- added ?: , pad:universal, F.Cu at (128.3, 135.3)
- added ?: , pad:universal, F.Cu at (97.8, 99.7)
- added ?: , pad:universal, F.Cu at (95.2, 99.7)
- added ?: , pad:universal, F.Cu at (95.2, 97.2)
- added ?: , pad:universal, F.Cu at (92.7, 99.7)
- added ?: , pad:universal, F.Cu at (95.2, 102.2)
- added ?: , pad:universal, F.Cu at (92.7, 97.2)
- added ?: , pad:universal, F.Cu at (92.7, 94.6)
- added ?: , pad:universal, F.Cu at (90.2, 94.6)
- added ?: , pad:universal, F.Cu at (95.2, 94.6)
- added ?: , pad:universal, F.Cu at (97.8, 94.6)
- added ?: , pad:universal, F.Cu at (135.9, 125.1)
- added ?: , pad:universal, F.Cu at (128.3, 137.8)
- added ?: , pad:universal, F.Cu at (110.5, 94.6)
- added ?: , pad:universal, F.Cu at (113.0, 94.6)
- added ?: , pad:universal, F.Cu at (113.0, 97.2)
- added ?: , pad:universal, F.Cu at (113.0, 99.7)
- added ?: , pad:universal, F.Cu at (108.0, 99.7)
- added ?: , pad:universal, F.Cu at (110.5, 99.7)
- added ?: , pad:universal, F.Cu at (110.5, 97.2)
- added ?: , pad:universal, F.Cu at (100.3, 107.3)
- added ?: , pad:universal, F.Cu at (102.9, 107.3)
- added ?: , pad:universal, F.Cu at (108.0, 104.8)
- added ?: , pad:universal, F.Cu at (130.8, 137.8)
- added ?: , pad:universal, F.Cu at (110.5, 104.8)
- added ?: , pad:universal, F.Cu at (110.5, 107.3)
- added ?: , pad:universal, F.Cu at (108.0, 107.3)
- added ?: , pad:universal, F.Cu at (105.4, 107.3)
- added ?: , pad:universal, F.Cu at (105.4, 104.8)
- added ?: , pad:universal, F.Cu at (102.9, 94.6)
- added ?: , pad:universal, F.Cu at (100.3, 99.7)
- added ?: , pad:universal, F.Cu at (100.3, 94.6)
- added ?: , pad:universal, F.Cu at (100.3, 97.2)
- added ?: , pad:universal, F.Cu at (108.0, 97.2)
- added ?: , pad:universal, F.Cu at (130.8, 135.3)
- added ?: , pad:universal, F.Cu at (105.4, 94.6)
- added ?: , pad:universal, F.Cu at (108.0, 94.6)
- added ?: , pad:universal, F.Cu at (105.4, 97.2)
- added ?: , pad:universal, F.Cu at (108.0, 102.2)
- added ?: , pad:universal, F.Cu at (113.0, 107.3)
- added ?: , pad:universal, F.Cu at (110.5, 102.2)
- added ?: , pad:universal, F.Cu at (113.0, 102.2)
- added ?: , pad:universal, F.Cu at (113.0, 104.8)
- added ?: , pad:universal, F.Cu at (100.3, 104.8)
- added ?: , pad:universal, F.Cu at (102.9, 104.8)
- added ?: , pad:universal, F.Cu at (128.3, 140.3)
- added ?: , pad:universal, F.Cu at (102.9, 102.2)
- added ?: , pad:universal, F.Cu at (105.4, 102.2)
- added ?: , pad:universal, F.Cu at (105.4, 99.7)
- added ?: , pad:universal, F.Cu at (102.9, 99.7)
- added ?: , pad:universal, F.Cu at (102.9, 97.2)
- added ?: , pad:universal, F.Cu at (100.3, 102.2)
- added ?: , pad:universal, F.Cu at (87.6, 97.2)
- added ?: , pad:universal, F.Cu at (90.2, 97.2)
- added ?: , pad:universal, F.Cu at (87.6, 94.6)
- added ?: , pad:universal, F.Cu at (97.8, 97.2)
- added ?: , pad:universal, F.Cu at (146.1, 127.6)
- added ?: , pad:universal, F.Cu at (120.7, 104.8)
- added ?: , pad:universal, F.Cu at (120.7, 107.3)
- added ?: , pad:universal, F.Cu at (118.1, 107.3)
- added ?: , pad:universal, F.Cu at (115.6, 104.8)
- added ?: , pad:universal, F.Cu at (115.6, 99.7)
- added ?: , pad:universal, F.Cu at (118.1, 104.8)
- added ?: , pad:universal, F.Cu at (115.6, 107.3)
- added ?: , pad:universal, F.Cu at (118.1, 102.2)
- added ?: , pad:universal, F.Cu at (115.6, 102.2)
- added ?: , pad:universal, F.Cu at (118.1, 99.7)
- added ?: , pad:universal, F.Cu at (143.5, 127.6)
- added ?: , pad:universal, F.Cu at (120.7, 97.2)
- added ?: , pad:universal, F.Cu at (120.7, 99.7)
- added ?: , pad:universal, F.Cu at (120.7, 102.2)
- added ?: , pad:universal, F.Cu at (179.1, 107.3)
- added ?: , pad:universal, F.Cu at (176.5, 107.3)
- added ?: , pad:universal, F.Cu at (181.6, 107.3)
- added ?: , pad:universal, F.Cu at (174.0, 107.3)
- added ?: , pad:universal, F.Cu at (171.4, 104.8)
- added ?: , pad:universal, F.Cu at (174.0, 104.8)
- added ?: , pad:universal, F.Cu at (171.4, 107.3)
- added ?: , pad:universal, F.Cu at (146.1, 130.2)
- added ?: , pad:universal, F.Cu at (171.4, 102.2)
- added ?: , pad:universal, F.Cu at (166.4, 102.2)
- added ?: , pad:universal, F.Cu at (168.9, 102.2)
- added ?: , pad:universal, F.Cu at (166.4, 107.3)
- added ?: , pad:universal, F.Cu at (168.9, 104.8)
- added ?: , pad:universal, F.Cu at (166.4, 104.8)
- added ?: , pad:universal, F.Cu at (168.9, 107.3)
- added ?: , pad:universal, F.Cu at (179.1, 94.6)
- added ?: , pad:universal, F.Cu at (181.6, 94.6)
- added ?: , pad:universal, F.Cu at (179.1, 97.2)
- added ?: , pad:universal, F.Cu at (143.5, 130.2)
- added ?: , pad:universal, F.Cu at (181.6, 97.2)
- added ?: , pad:universal, F.Cu at (181.6, 99.7)
- added ?: , pad:universal, F.Cu at (179.1, 99.7)
- added ?: , pad:universal, F.Cu at (181.6, 102.2)
- added ?: , pad:universal, F.Cu at (176.5, 104.8)
- added ?: , pad:universal, F.Cu at (179.1, 102.2)
- added ?: , pad:universal, F.Cu at (179.1, 104.8)
- added ?: , pad:universal, F.Cu at (181.6, 104.8)
- added ?: , pad:universal, F.Cu at (174.0, 102.2)
- added ?: , pad:universal, F.Cu at (176.5, 102.2)
- added ?: , pad:universal, F.Cu at (143.5, 132.7)
- added ?: , pad:universal, F.Cu at (174.0, 99.7)
- added ?: , pad:universal, F.Cu at (176.5, 99.7)
- added ?: , pad:universal, F.Cu at (151.1, 94.6)
- added ?: , pad:universal, F.Cu at (148.6, 94.6)
- added ?: , pad:universal, F.Cu at (151.1, 97.2)
- added ?: , pad:universal, F.Cu at (166.4, 99.7)
- added ?: , pad:universal, F.Cu at (168.9, 99.7)
- added ?: , pad:universal, F.Cu at (163.8, 99.7)
- added ?: , pad:universal, F.Cu at (166.4, 97.2)
- added ?: , pad:universal, F.Cu at (163.8, 97.2)
- added ?: , pad:universal, F.Cu at (146.1, 132.7)
- added ?: , pad:universal, F.Cu at (163.8, 94.6)
- added ?: , pad:universal, F.Cu at (166.4, 94.6)
- added ?: , pad:universal, F.Cu at (168.9, 97.2)
- added ?: , pad:universal, F.Cu at (168.9, 94.6)
- added ?: , pad:universal, F.Cu at (171.4, 99.7)
- added ?: , pad:universal, F.Cu at (174.0, 97.2)
- added ?: , pad:universal, F.Cu at (176.5, 94.6)
- added ?: , pad:universal, F.Cu at (171.4, 97.2)
- added ?: , pad:universal, F.Cu at (176.5, 97.2)
- added ?: , pad:universal, F.Cu at (174.0, 94.6)
- added ?: , pad:universal, F.Cu at (133.3, 125.1)
- added ?: , pad:universal, F.Cu at (146.1, 137.8)
- added ?: , pad:universal, F.Cu at (171.4, 94.6)
- added ?: , pad:universal, F.Cu at (148.6, 102.2)
- added ?: , pad:universal, F.Cu at (151.1, 102.2)
- added ?: , pad:universal, F.Cu at (148.6, 99.7)
- added ?: , pad:universal, F.Cu at (151.1, 99.7)
- added ?: , pad:universal, F.Cu at (163.8, 104.8)
- added ?: , pad:universal, F.Cu at (161.3, 104.8)
- added ?: , pad:universal, F.Cu at (161.3, 107.3)
- added ?: , pad:universal, F.Cu at (163.8, 102.2)
- added ?: , pad:universal, F.Cu at (161.3, 102.2)
- added ?: , pad:universal, F.Cu at (146.1, 135.3)
- added ?: , pad:universal, F.Cu at (163.8, 107.3)
- added ?: , pad:universal, F.Cu at (148.6, 104.8)
- added ?: , pad:universal, F.Cu at (151.1, 107.3)
- added ?: , pad:universal, F.Cu at (151.1, 104.8)
- added ?: , pad:universal, F.Cu at (148.6, 107.3)
- added ?: , pad:universal, F.Cu at (158.8, 102.2)
- added ?: , pad:universal, F.Cu at (158.8, 97.2)
- added ?: , pad:universal, F.Cu at (158.8, 99.7)
- added ?: , pad:universal, F.Cu at (161.3, 99.7)
- added ?: , pad:universal, F.Cu at (161.3, 97.2)
- added ?: , pad:universal, F.Cu at (146.1, 140.3)
- added ?: , pad:universal, F.Cu at (148.6, 97.2)
- added ?: , pad:universal, F.Cu at (153.7, 99.7)
- added ?: , pad:universal, F.Cu at (156.2, 99.7)
- added ?: , pad:universal, F.Cu at (153.7, 97.2)
- added ?: , pad:universal, F.Cu at (153.7, 94.6)
- added ?: , pad:universal, F.Cu at (156.2, 97.2)
- added ?: , pad:universal, F.Cu at (156.2, 94.6)
- added ?: , pad:universal, F.Cu at (153.7, 107.3)
- added ?: , pad:universal, F.Cu at (153.7, 104.8)
- added ?: , pad:universal, F.Cu at (153.7, 102.2)
- added ?: , pad:universal, F.Cu at (135.9, 137.8)
- added ?: , pad:universal, F.Cu at (156.2, 107.3)
- added ?: , pad:universal, F.Cu at (158.8, 107.3)
- added ?: , pad:universal, F.Cu at (158.8, 104.8)
- added ?: , pad:universal, F.Cu at (156.2, 104.8)
- added ?: , pad:universal, F.Cu at (156.2, 102.2)
- added ?: , pad:universal, F.Cu at (158.8, 94.6)
- added ?: , pad:universal, F.Cu at (161.3, 94.6)
- added ?: , pad:universal, F.Cu at (141.0, 155.6)
- added ?: , pad:universal, F.Cu at (141.0, 153.0)
- added ?: , pad:universal, F.Cu at (141.0, 150.5)
- added ?: , pad:universal, F.Cu at (133.3, 135.3)
- added ?: , pad:universal, F.Cu at (143.5, 150.5)
- added ?: , pad:universal, F.Cu at (138.4, 155.6)
- added ?: , pad:universal, F.Cu at (138.4, 153.0)
- added ?: , pad:universal, F.Cu at (138.4, 150.5)
- added ?: , pad:universal, F.Cu at (135.9, 150.5)
- added ?: , pad:universal, F.Cu at (135.9, 155.6)
- added ?: , pad:universal, F.Cu at (133.3, 155.6)
- added ?: , pad:universal, F.Cu at (133.3, 150.5)
- added ?: , pad:universal, F.Cu at (133.3, 153.0)
- added ?: , pad:universal, F.Cu at (135.9, 153.0)
- added ?: , pad:universal, F.Cu at (133.3, 140.3)
- added ?: , pad:universal, F.Cu at (143.5, 155.6)
- added ?: , pad:universal, F.Cu at (146.1, 155.6)
- added ?: , pad:universal, F.Cu at (146.1, 150.5)
- added ?: , pad:universal, F.Cu at (146.1, 153.0)
- added ?: , pad:universal, F.Cu at (143.5, 153.0)
- added ?: , pad:universal, F.Cu at (148.6, 150.5)
- added ?: , pad:universal, F.Cu at (181.6, 150.5)
- added ?: , pad:universal, F.Cu at (179.1, 150.5)
- added ?: , pad:universal, F.Cu at (176.5, 150.5)
- added ?: , pad:universal, F.Cu at (171.4, 150.5)
- added ?: , pad:universal, F.Cu at (135.9, 140.3)
- added ?: , pad:universal, F.Cu at (163.8, 153.0)
- added ?: , pad:universal, F.Cu at (163.8, 150.5)
- added ?: , pad:universal, F.Cu at (166.4, 150.5)
- added ?: , pad:universal, F.Cu at (168.9, 150.5)
- added ?: , pad:universal, F.Cu at (166.4, 155.6)
- added ?: , pad:universal, F.Cu at (163.8, 155.6)
- added ?: , pad:universal, F.Cu at (168.9, 153.0)
- added ?: , pad:universal, F.Cu at (166.4, 153.0)
- added ?: , pad:universal, F.Cu at (168.9, 155.6)
- added ?: , pad:universal, F.Cu at (174.0, 155.6)
- added ?: , pad:universal, F.Cu at (135.9, 135.3)
- added ?: , pad:universal, F.Cu at (171.4, 153.0)
- added ?: , pad:universal, F.Cu at (174.0, 153.0)
- added ?: , pad:universal, F.Cu at (171.4, 155.6)
- added ?: , pad:universal, F.Cu at (174.0, 150.5)
- added ?: , pad:universal, F.Cu at (179.1, 155.6)
- added ?: , pad:universal, F.Cu at (181.6, 155.6)
- added ?: , pad:universal, F.Cu at (176.5, 155.6)
- added ?: , pad:universal, F.Cu at (176.5, 153.0)
- added ?: , pad:universal, F.Cu at (179.1, 153.0)
- added ?: , pad:universal, F.Cu at (181.6, 153.0)
- added ?: , pad:universal, F.Cu at (133.3, 137.8)
- added ?: , pad:universal, F.Cu at (153.7, 155.6)
- added ?: , pad:universal, F.Cu at (148.6, 155.6)
- added ?: , pad:universal, F.Cu at (148.6, 153.0)
- added ?: , pad:universal, F.Cu at (151.1, 155.6)
- added ?: , pad:universal, F.Cu at (151.1, 153.0)
- added ?: , pad:universal, F.Cu at (153.7, 153.0)
- added ?: , pad:universal, F.Cu at (153.7, 150.5)
- added ?: , pad:universal, F.Cu at (151.1, 150.5)
- added ?: , pad:universal, F.Cu at (156.2, 155.6)
- added ?: , pad:universal, F.Cu at (158.8, 155.6)
- added ?: , pad:universal, F.Cu at (143.5, 137.8)
- added ?: , pad:universal, F.Cu at (161.3, 153.0)
- added ?: , pad:universal, F.Cu at (161.3, 155.6)
- added ?: , pad:universal, F.Cu at (158.8, 153.0)
- added ?: , pad:universal, F.Cu at (156.2, 153.0)
- added ?: , pad:universal, F.Cu at (156.2, 150.5)
- added ?: , pad:universal, F.Cu at (158.8, 150.5)
- added ?: , pad:universal, F.Cu at (161.3, 150.5)
- added ?: , pad:universal, F.Cu at (100.3, 153.0)
- added ?: , pad:universal, F.Cu at (100.3, 155.6)
- added ?: , pad:universal, F.Cu at (102.9, 150.5)
- added ?: , pad:universal, F.Cu at (141.0, 125.1)
- added ?: , pad:universal, F.Cu at (138.4, 137.8)
- added ?: , pad:universal, F.Cu at (100.3, 150.5)
- added ?: , pad:universal, F.Cu at (108.0, 153.0)
- added ?: , pad:universal, F.Cu at (110.5, 150.5)
- added ?: , pad:universal, F.Cu at (110.5, 153.0)
- added ?: , pad:universal, F.Cu at (113.0, 155.6)
- added ?: , pad:universal, F.Cu at (110.5, 155.6)
- added ?: , pad:universal, F.Cu at (108.0, 150.5)
- added ?: , pad:universal, F.Cu at (108.0, 155.6)
- added ?: , pad:universal, F.Cu at (105.4, 155.6)
- added ?: , pad:universal, F.Cu at (105.4, 153.0)
- added ?: , pad:universal, F.Cu at (141.0, 135.3)
- added ?: , pad:universal, F.Cu at (105.4, 150.5)
- added ?: , pad:universal, F.Cu at (102.9, 155.6)
- added ?: , pad:universal, F.Cu at (102.9, 153.0)
- added ?: , pad:universal, F.Cu at (130.8, 155.6)
- added ?: , pad:universal, F.Cu at (130.8, 153.0)
- added ?: , pad:universal, F.Cu at (128.3, 153.0)
- added ?: , pad:universal, F.Cu at (128.3, 155.6)
- added ?: , pad:universal, F.Cu at (130.8, 150.5)
- added ?: , pad:universal, F.Cu at (128.3, 150.5)
- added ?: , pad:universal, F.Cu at (125.7, 155.6)
- added ?: , pad:universal, F.Cu at (141.0, 137.8)
- added ?: , pad:universal, F.Cu at (125.7, 153.0)
- added ?: , pad:universal, F.Cu at (123.2, 155.6)
- added ?: , pad:universal, F.Cu at (123.2, 153.0)
- added ?: , pad:universal, F.Cu at (125.7, 150.5)
- added ?: , pad:universal, F.Cu at (118.1, 155.6)
- added ?: , pad:universal, F.Cu at (120.7, 153.0)
- added ?: , pad:universal, F.Cu at (120.7, 155.6)
- added ?: , pad:universal, F.Cu at (118.1, 153.0)
- added ?: , pad:universal, F.Cu at (115.6, 155.6)
- added ?: , pad:universal, F.Cu at (118.1, 150.5)
- added ?: , pad:universal, F.Cu at (143.5, 135.3)
- added ?: , pad:universal, F.Cu at (115.6, 153.0)
- added ?: , pad:universal, F.Cu at (115.6, 150.5)
- added ?: , pad:universal, F.Cu at (123.2, 150.5)
- added ?: , pad:universal, F.Cu at (120.7, 150.5)
- added ?: , pad:universal, F.Cu at (113.0, 153.0)
- added ?: , pad:universal, F.Cu at (113.0, 150.5)
- added ?: , pad:universal, F.Cu at (92.7, 153.0)
- added ?: , pad:universal, F.Cu at (97.8, 150.5)
- added ?: , pad:universal, F.Cu at (97.8, 153.0)
- added ?: , pad:universal, F.Cu at (97.8, 155.6)
- added ?: , pad:universal, F.Cu at (138.4, 135.3)
- added ?: , pad:universal, F.Cu at (92.7, 155.6)
- added ?: , pad:universal, F.Cu at (95.2, 153.0)
- added ?: , pad:universal, F.Cu at (95.2, 150.5)
- added ?: , pad:universal, F.Cu at (95.2, 155.6)
- added ?: , pad:universal, F.Cu at (90.2, 155.6)
- added ?: , pad:universal, F.Cu at (92.7, 150.5)
- added ?: , pad:universal, F.Cu at (87.6, 150.5)
- added ?: , pad:universal, F.Cu at (87.6, 155.6)
- added ?: , pad:universal, F.Cu at (90.2, 150.5)
- added ?: , pad:universal, F.Cu at (87.6, 153.0)
- added ?: , pad:universal, F.Cu at (143.5, 140.3)
- added ?: , pad:universal, F.Cu at (90.2, 153.0)
- added ?: , pad:universal, F.Cu at (141.0, 148.0)
- added ?: , pad:universal, F.Cu at (138.4, 148.0)
- added ?: , pad:universal, F.Cu at (135.9, 148.0)
- added ?: , pad:universal, F.Cu at (133.3, 148.0)
- added ?: , pad:universal, F.Cu at (143.5, 148.0)
- added ?: , pad:universal, F.Cu at (146.1, 148.0)
- added ?: , pad:universal, F.Cu at (130.8, 148.0)
- added ?: , pad:universal, F.Cu at (128.3, 148.0)
- added ?: , pad:universal, F.Cu at (125.7, 148.0)
- added ?: , pad:universal, F.Cu at (141.0, 140.3)
- added ?: , pad:universal, F.Cu at (123.2, 148.0)
- added ?: , pad:universal, F.Cu at (141.0, 145.4)
- added ?: , pad:universal, F.Cu at (138.4, 145.4)
- added ?: , pad:universal, F.Cu at (135.9, 145.4)
- added ?: , pad:universal, F.Cu at (133.3, 145.4)
- added ?: , pad:universal, F.Cu at (143.5, 145.4)
- added ?: , pad:universal, F.Cu at (146.1, 145.4)
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Connections:
- U2 pad 19: (no net) -> Net-(J26-Pad1)
- U2 pad 20: (no net) -> Net-(J25-Pad1)
Routing:
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- added copper zone on F.Cu, net GND
Other:
- board size 100 x 100 mm -> 105 x 100 mm
- net class Default: via_dia 0.6 -> 0.5
- board text added: "LPC1114 Universal @JP3CYC"
- board text added: "SWCLK"
- board text added: "SWDIO"
- board text added: "Xin"
- board text added: "Xout"
- board text added: "dp10"
- board text added: "dp11"
- board text added: "dp13"
- board text added: "dp14"
- board text added: "dp15"
- board text added: "dp16"
- board text added: "dp17"
- board text added: "dp23"
- board text added: "dp25"
- board text added: "dp26"
- board text added: "dp27"
- board text added: "dp28"
- board text added: "dp4"
- board text added: "dp5"
- board text added: "dp6"
- board text added: "dp9"
- board text added: "~~dp1"
- board text added: "~~dp18"
- board text added: "~~dp2"
- board text added: "~~dp24"

Commit message: 製造ファイル作成
Parts:
- added D1: LED, LEDs:LED_D3.0mm, F.Cu at (106.7, 80.6)
- added R1: R, Resistors_SMD:R_0603_HandSoldering, F.Cu at (105.6, 85.1)
- U2: value lpc1114fdh28 -> lpc1114fn28
Connections:
- J23 pad 2: (no net) -> Net-(J23-Pad2)
- J23 pad 3: +5V -> +3V3
- J23 pad 6: (no net) -> Net-(J23-Pad6)
- J25 pad 1: Net-(J25-Pad1) -> Net-(J23-Pad2)
- J26 pad 1: Net-(J26-Pad1) -> Net-(J23-Pad6)
- U2 pad 19: Net-(J26-Pad1) -> Net-(J23-Pad6)
- U2 pad 20: Net-(J25-Pad1) -> Net-(J23-Pad2)
Routing:
- net Net-(J23-Pad2): track 0.00 -> 55.9 mm, vias 0 -> 1
- net +3V3: track 82.4 -> 133.8 mm
- net +5V: track 79.0 -> 31.3 mm
- net Net-(J23-Pad6): track 0.00 -> 43.3 mm
- net GND: track 124.5 -> 145.3 mm
- net Net-(J26-Pad1): track 7.73 -> 0.00 mm
- net Net-(J25-Pad1): track 6.95 -> 0.00 mm
- net Net-(D1-Pad2): track 0.00 -> 4.59 mm
- net Net-(J21-Pad1): track 57.0 -> 53.9 mm
- net Net-(J22-Pad1): track 56.8 -> 55.1 mm
- net Net-(J17-Pad1): track 7.34 -> 8.14 mm
Other:
- board text added: "3.3V"
- board text added: "<RXD"
- board text added: ">TXD"
- board text added: "DTR"
- board text added: "GND"
- board text added: "RTS"
