File: mbed_lpc1114.sch (KiCad schematic (older format))
At the start: 32 parts, among them J1 CONN_01X01, J10 CONN_01X01, J11 CONN_01X01, J12 CONN_01X01, J13 CONN_01X01, J14 CONN_01X01, J15 CONN_01X01, J16 CONN_01X01, J17 CONN_01X01, J18 CONN_01X01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

Commit message: 完成
Parts:
- added J25, J26: CONN_01X01, pad:universal, symbol CONN_01X01
- J24: footprint Connect:JACK_ALIM -> Connectors:BARREL_JACK
- U1: footprint mylib:7805 -> TO_SOT_Packages_SMD:TO-252-3_TabPin2
- U2: footprint Housings_DIP:DIP-28_W15.24mm_LongPads -> Housings_SSOP:TSSOP-28_4.4x9.7mm_Pitch0.65mm
Connections:
- net at U2.19 (XTAOUT): now also J26.1 (P1)
- net at U2.20 (XTALIN): now also J25.1 (P1)
- no-connect marks 4 -> 2
Changed lines of the file:
@@
 F 0 "U1" H 4950 1854 50  0000 C CNN
 F 1 "7803" H 4800 2250 50  0000 C CNN
-F 2 "mylib:7805" H 4800 2050 50  0001 C CNN
+F 2 "TO_SOT_Packages_SMD:TO-252-3_TabPin2" H 4800 2050 50  0001 C CNN
 F 3 "" H 4800 2050 50  0001 C CNN
 	1    4800 2050
@@
 Wire Wire Line
 	7800 4750 7800 4700
-NoConn ~ 6650 4700
-NoConn ~ 6650 4600
 $Comp
 L +3.3V #PWR07
@@
 F 3 "" H 7800 4700 50  0001 C CNN
 	1    7800 4700
-	1    0    0    -1
-$EndComp
-$Comp
-L lpc1114fn28 U2
-U 1 1 5904732E
-P 5800 4450
-F 0 "U2" H 6350 5300 60  0000 C CNN
-F 1 "lpc1114fn28" H 5800 5300 60  0000 C CNN
-F 2 "Housings_DIP:DIP-28_W15.24mm_LongPads" H 5800 4450 60  0001 C CNN
-F 3 "" H 5800 4450 60  0001 C CNN
-	1    5800 4450
 	1    0    0    -1
 $EndComp
@@
 F 0 "J24" H 2200 2445 50  0000 C CNN
 F 1 "BARREL_JACK" H 2200 2095 50  0000 C CNN
-F 2 "Connect:JACK_ALIM" H 2200 2250 50  0001 C CNN
+F 2 "Connectors:BARREL_JACK" H 2200 2250 50  0001 C CNN
 F 3 "" H 2200 2250 50  0001 C CNN
 	1    2200 2250
@@
 Connection ~ 2500 2150
 Connection ~ 2500 2350
+$Comp
+L lpc1114fn28 U2
+U 1 1 5904732E
+P 5800 4450
+F 0 "U2" H 6350 5300 60  0000 C CNN
+F 1 "lpc1114fn28" H 5800 5300 60  0000 C CNN
+F 2 "Housings_SSOP:TSSOP-28_4.4x9.7mm_Pitch0.65mm" H 5800 4450 60  0001 C CNN
+F 3 "" H 5800 4450 60  0001 C CNN
+	1    5800 4450
+	1    0    0    -1
+$EndComp
+$Comp
+L CONN_01X01 J25
+U 1 1 596221CD
+P 6850 4600
+F 0 "J25" H 6950 4600 50  0000 C CNN
+F 1 "CONN_01X01" V 6950 4600 50  0001 C CNN
+F 2 "pad:universal" H 6850 4600 50  0001 C CNN
+F 3 "" H 6850 4600 50  0001 C CNN
+	1    6850 4600
+	1    0    0    1
+$EndComp
+$Comp
+L CONN_01X01 J26
+U 1 1 59622250
+P 6850 4700
+F 0 "J26" H 6950 4700 50  0000 C CNN
+F 1 "CONN_01X01" V 6950 4700 50  0001 C CNN
+F 2 "pad:universal" H 6850 4700 50  0001 C CNN
+F 3 "" H 6850 4700 50  0001 C CNN
+	1    6850 4700
+	1    0    0    1
+$EndComp
 $EndSCHEMATC

Commit message: 製造ファイル作成
Parts:
- added D1: LED, LEDs:LED_D3.0mm, symbol LED
- added R1: R, Resistors_SMD:R_0603_HandSoldering, symbol R
Connections:
- net +3V3: now also J23.3 (P3), R1.1
- net +5V: no longer J23.3 (P3)
- net GND: now also D1.1 (K)
- net at J26.1 (P1), U2.19 (XTAOUT): now also J23.6 (P6)
- net at J25.1 (P1), U2.20 (XTALIN): now also J23.2 (P2)
- new net: D1.2 (A), R1.2
- no-connect marks 2 -> 0
Other:
- moved on the sheet: C6
Changed lines of the file:
@@
 L GND #PWR04
 U 1 1 5904484A
-P 7500 4450
-F 0 "#PWR04" H 7500 4200 50  0001 C CNN
-F 1 "GND" H 7500 4300 50  0000 C CNN
-F 2 "" H 7500 4450 50  0001 C CNN
-F 3 "" H 7500 4450 50  0001 C CNN
-	1    7500 4450
+P 7800 4450
+F 0 "#PWR04" H 7800 4200 50  0001 C CNN
+F 1 "GND" H 7800 4300 50  0000 C CNN
+F 2 "" H 7800 4450 50  0001 C CNN
+F 3 "" H 7800 4450 50  0001 C CNN
+	1    7800 4450
 	1    0    0    -1
 $EndComp
@@
 L C C6
 U 1 1 590448CD
-P 7300 4550
-F 0 "C6" H 7325 4650 50  0000 L CNN
-F 1 "1uF" H 7325 4450 50  0000 L CNN
-F 2 "Capacitors_SMD:C_0603_HandSoldering" H 7338 4400 50  0001 C CNN
-F 3 "" H 7300 4550 50  0001 C CNN
-	1    7300 4550
+P 7600 4550
+F 0 "C6" H 7625 4650 50  0000 L CNN
+F 1 "1uF" H 7625 4450 50  0000 L CNN
+F 2 "Capacitors_SMD:C_0603_HandSoldering" H 7638 4400 50  0001 C CNN
+F 3 "" H 7600 4550 50  0001 C CNN
+	1    7600 4550
 	1    0    0    -1
 $EndComp
@@
 Connection ~ 5700 2000
 Wire Wire Line
-	6650 4400 7100 4400
-Wire Wire Line
-	7100 4400 7100 4350
-Wire Wire Line
-	7300 4750 7300 4700
-Wire Wire Line
-	7300 4400 7300 4350
-Wire Wire Line
-	7100 4350 7500 4350
-Connection ~ 7300 4750
-Connection ~ 7300 4350
+	6650 4400 7400 4400
+Wire Wire Line
+	7400 4400 7400 4350
+Wire Wire Line
+	7600 4750 7600 4700
+Wire Wire Line
+	7600 4400 7600 4350
+Wire Wire Line
+	7400 4350 7800 4350
+Connection ~ 7600 4750
+Connection ~ 7600 4350
 Wire Wire Line
 	4950 4500 4000 4500
@@
 Connection ~ 3800 4650
 Wire Wire Line
-	7500 4350 7500 4450
-Wire Wire Line
-	7800 4750 7800 4700
+	7800 4350 7800 4450
+Wire Wire Line
+	8100 4750 8100 4700
 $Comp
 L +3.3V #PWR07
 U 1 1 59057C94
-P 7800 4700
-F 0 "#PWR07" H 7800 4550 50  0001 C CNN
-F 1 "+3.3V" H 7800 4840 50  0000 C CNN
-F 2 "" H 7800 4700 50  0001 C CNN
-F 3 "" H 7800 4700 50  0001 C CNN
-	1    7800 4700
-	1    0    0    -1
-$EndComp
-Wire Wire Line
-	6650 4500 7000 4500
-Wire Wire Line
-	7000 4500 7000 4750
-Wire Wire Line
-	7000 4750 7800 4750
+P 8100 4700
+F 0 "#PWR07" H 8100 4550 50  0001 C CNN
+F 1 "+3.3V" H 8100 4840 50  0000 C CNN
+F 2 "" H 8100 4700 50  0001 C CNN
+F 3 "" H 8100 4700 50  0001 C CNN
+	1    8100 4700
+	1    0    0    -1
+$EndComp
+Wire Wire Line
+	6650 4500 7400 4500
+Wire Wire Line
+	7400 4500 7400 4750
+Wire Wire Line
+	7400 4750 8100 4750
 $Comp
 L CONN_01X01 J1
@@
 $EndComp
 $Comp
-L +5V #PWR09
-U 1 1 59509D04
-P 7550 5700
-F 0 "#PWR09" H 7550 5550 50  0001 C CNN
-F 1 "+5V" H 7550 5840 50  0000 C CNN
-F 2 "" H 7550 5700 50  0001 C CNN
-F 3 "" H 7550 5700 50  0001 C CNN
-	1    7550 5700
-	0    -1   -1   0
-$EndComp
-NoConn ~ 7550 5600
-NoConn ~ 7550 6000
-$Comp
 L BARREL_JACK J24
 U 1 1 5950D2CD
@@
 $EndComp
 $Comp
-L GND #PWR010
+L GND #PWR09
 U 1 1 5950D614
 P 2750 2400
-F 0 "#PWR010" H 2750 2150 50  0001 C CNN
+F 0 "#PWR09" H 2750 2150 50  0001 C CNN
 F 1 "GND" H 2750 2250 50  0000 C CNN
 F 2 "" H 2750 2400 50  0001 C CNN
@@
 $EndComp
 $Comp
-L +5V #PWR011
+L +5V #PWR010
 U 1 1 5950D67F
 P 2750 2150
-F 0 "#PWR011" H 2750 2000 50  0001 C CNN
+F 0 "#PWR010" H 2750 2000 50  0001 C CNN
 F 1 "+5V" H 2750 2290 50  0000 C CNN
 F 2 "" H 2750 2150 50  0001 C CNN
@@
 	3800 4650 4000 4650
 $Comp
-L PWR_FLAG #FLG012
+L PWR_FLAG #FLG011
 U 1 1 59510BFD
 P 2500 2100
-F 0 "#FLG012" H 2500 2175 50  0001 C CNN
+F 0 "#FLG011" H 2500 2175 50  0001 C CNN
 F 1 "PWR_FLAG" H 2500 2250 50  0000 C CNN
 F 2 "" H 2500 2100 50  0001 C CNN
@@
 $EndComp
 $Comp
-L PWR_FLAG #FLG013
+L PWR_FLAG #FLG012
 U 1 1 59510CD4
 P 2500 2450
-F 0 "#FLG013" H 2500 2525 50  0001 C CNN
+F 0 "#FLG012" H 2500 2525 50  0001 C CNN
 F 1 "PWR_FLAG" H 2500 2600 50  0000 C CNN
 F 2 "" H 2500 2450 50  0001 C CNN
@@
 	1    0    0    1
 $EndComp
+$Comp
+L R R1
+U 1 1 5970B7F4
+P 6450 2150
+F 0 "R1" V 6530 2150 50  0000 C CNN
+F 1 "R" V 6450 2150 50  0000 C CNN
+F 2 "Resistors_SMD:R_0603_HandSoldering" V 6380 2150 50  0001 C CNN
+F 3 "" H 6450 2150 50  0001 C CNN
+	1    6450 2150
+	1    0    0    -1
+$EndComp
+$Comp
+L LED D1
+U 1 1 5970B85D
+P 6450 2450
+F 0 "D1" H 6450 2550 50  0000 C CNN
+F 1 "LED" H 6450 2350 50  0000 C CNN
+F 2 "LEDs:LED_D3.0mm" H 6450 2450 50  0001 C CNN
+F 3 "" H 6450 2450 50  0001 C CNN
+	1    6450 2450
+	0    -1   -1   0
+$EndComp
+$Comp
+L GND #PWR013
+U 1 1 5970B8E6
+P 6450 2600
+F 0 "#PWR013" H 6450 2350 50  0001 C CNN
+F 1 "GND" H 6450 2450 50  0000 C CNN
+F 2 "" H 6450 2600 50  0001 C CNN
+F 3 "" H 6450 2600 50  0001 C CNN
+	1    6450 2600
+	1    0    0    -1
+$EndComp
+Wire Wire Line
+	7100 6000 7550 6000
+Wire Wire Line
+	7350 5600 7550 5600
+Wire Wire Line
+	7350 4650 7350 5600
+Wire Wire Line
+	7350 4650 6650 4650
+Wire Wire Line
+	6650 4650 6650 4600
+Connection ~ 6650 4700
+Connection ~ 6650 4600
+Wire Wire Line
+	6650 4700 6650 4750
+Wire Wire Line
+	6650 4750 7100 4750
+Wire Wire Line
+	7100 4750 7100 6000
+$Comp
+L +3.3V #PWR014
+U 1 1 59723C81
+P 7550 5700
+F 0 "#PWR014" H 7550 5550 50  0001 C CNN
+F 1 "+3.3V" H 7550 5840 50  0000 C CNN
+F 2 "" H 7550 5700 50  0001 C CNN
+F 3 "" H 7550 5700 50  0001 C CNN
+	1    7550 5700
+	0    -1   -1   0
+$EndComp
+$Comp
+L +3.3V #PWR015
+U 1 1 59724277
+P 6450 2000
+F 0 "#PWR015" H 6450 1850 50  0001 C CNN
+F 1 "+3.3V" H 6450 2140 50  0000 C CNN
+F 2 "" H 6450 2000 50  0001 C CNN
+F 3 "" H 6450 2000 50  0001 C CNN
+	1    6450 2000
+	1    0    0    -1
+$EndComp
 $EndSCHEMATC
